Commit message: [week02] models: 뷰어 확인에서 발견한 베이스-link1 충돌 수정 (base_link collision 제거)
어깨가 수평에서 멈추던 원인(접촉 1개)을 제거 → 하한 +90°까지 낙하 확인.
수정 전 뷰어 캡처, 낙하 CSV 갱신, 임포트 체크리스트 A6-2 추가.

Co-Authored-By: Claude Opus 5.5 <noreply@anthropic.com>
Claude-Session: https://claude.ai/code/session_01H2kByPNPXvMp7PWKcwQaQh

File: members/park-jongjin/week02/models/two_link_arm.urdf (robot description, URDF)
Before this commit: robot two_link_arm, 4 links, 3 joints
Links:
- link base_link: geometry visual cylinder length=0.10 radius=0.05
