Commit message: [week04] 함태훈 검증 반영 v0.1: RI85 출력측 = output-v1+ring2+cover plate1(elbow 2.2677 kg), left yaw +z, 축 규약 안(§6), 보고서 · 로그 갱신
Co-Authored-By: Claude Opus 5.5 <noreply@anthropic.com>
Claude-Session: https://claude.ai/code/session_015MVFLpu6hAhyrX1HywEtmx

File: b1/models/v0/urdf/b1_humanoid_skeleton.urdf (robot description, URDF)
Before this commit: robot b1_humanoid_skeleton, 13 links, 12 joints
Links:
- link left_elbow_link: mass 2.1425 -> 2.2677
- link right_elbow_link: mass 2.1425 -> 2.2677
- link torso_link: mass 12.741 -> 12.491
Joints:
- joint left_shoulder_yaw_joint: axis 0 0 -1 -> 0 0 1
- joint right_shoulder_yaw_joint: axis 0 0 1 -> 0 0 -1

File: b1/models/v0/urdf/b1_humanoid_v0.urdf (robot description, URDF)
Before this commit: robot b1_humanoid_v0, 13 links, 12 joints
Links:
- link left_elbow_link: mass 2.1425 -> 2.2677
- link right_elbow_link: mass 2.1425 -> 2.2677
- link torso_link: mass 12.741 -> 12.491
Joints:
- joint left_shoulder_yaw_joint: axis 0 0 -1 -> 0 0 1
- joint right_shoulder_yaw_joint: axis 0 0 1 -> 0 0 -1

Commit message: [week04] 팀장 10/14 회신 반영: REP 103 + CAD→base 고정 변환(cad_frame), 영점 = 팔 내림·팔꿈치 전방 굽힘(yaw origin rpy), joint 원점 검증표 + B2 부호표 초안, A1 확인 요청 그림, 보고서 부록 D
Co-Authored-By: Claude Opus 5.5 <noreply@anthropic.com>
Claude-Session: https://claude.ai/code/session_015MVFLpu6hAhyrX1HywEtmx

File: b1/models/v0/urdf/b1_humanoid_skeleton.urdf (robot description, URDF)
Before this commit: robot b1_humanoid_skeleton, 13 links, 12 joints
Links:
- added link cad_frame, mass 0.001
Joints:
- added joint cad_frame_joint: type fixed, parent torso_link, child cad_frame, origin xyz=0 0.11815 0 rpy=1.5708 0 1.5708
- joint left_shoulder_yaw_joint: origin xyz=0 0 -0.1823 rpy=0 0 0 -> xyz=0 0 -0.1823 rpy=0 0 -1.5708
- joint right_shoulder_yaw_joint: origin xyz=0 0 -0.1823 rpy=0 0 0 -> xyz=0 0 -0.1823 rpy=0 0 1.5708

File: b1/models/v0/urdf/b1_humanoid_v0.urdf (robot description, URDF)
Before this commit: robot b1_humanoid_v0, 13 links, 12 joints
Links:
- added link cad_frame, mass 0.001
Joints:
- added joint cad_frame_joint: type fixed, parent torso_link, child cad_frame, origin xyz=0 0.11815 0 rpy=1.5708 0 1.5708
- joint left_shoulder_yaw_joint: origin xyz=0 0 -0.1823 rpy=0 0 0 -> xyz=0 0 -0.1823 rpy=0 0 -1.5708
- joint right_shoulder_yaw_joint: origin xyz=0 0 -0.1823 rpy=0 0 0 -> xyz=0 0 -0.1823 rpy=0 0 1.5708

Commit message: [week04] v0 = 함태훈 메시·inertial(f9c9eff) + 박종진 골격 통합: 링크 원점 차(축 방향 17~22 mm) 평행이동 보정, 74.10 kg, 체크리스트 25 OK, 캡처 · 보고서 갱신
Co-Authored-By: Claude Opus 5.5 <noreply@anthropic.com>
Claude-Session: https://claude.ai/code/session_015MVFLpu6hAhyrX1HywEtmx

File: b1/models/v0/urdf/b1_humanoid_skeleton.urdf (robot description, URDF)
Before this commit: robot b1_humanoid_skeleton, 14 links, 13 joints
Links:
- link left_shoulder_pitch_link: mass 4.6099 -> 4.3963
- link left_shoulder_roll_link: mass 4.3831 -> 4.1696
- link left_shoulder_yaw_link: mass 3.55 -> 3.3364
- link right_shoulder_pitch_link: mass 4.6099 -> 4.3963
- link right_shoulder_roll_link: mass 4.3831 -> 4.1696
- link right_shoulder_yaw_link: mass 3.55 -> 3.3364
- link torso_link: mass 12.491 -> 12.063

File: b1/models/v0/urdf/b1_humanoid_v0.urdf (robot description, URDF)
Before this commit: robot b1_humanoid_v0, 14 links, 13 joints
Links:
- link left_shoulder_pitch_link: mass 4.6099 -> 4.3963
- link left_shoulder_roll_link: mass 4.3831 -> 4.1696
- link left_shoulder_yaw_link: mass 3.55 -> 3.3364
- link right_shoulder_pitch_link: mass 4.6099 -> 4.3963
- link right_shoulder_roll_link: mass 4.3831 -> 4.1696
- link right_shoulder_yaw_link: mass 3.55 -> 3.3364
- link torso_link: mass 12.491 -> 12.063
