Commit message: [week06] A2 구동기 사양 반영 + 중력보상 기본 on + 메시 visual/collision 분리
- inputs/a2_actuators.json: case a2_doc(어깨 TQ armature 0.219 · 피크 381.7, 팔꿈치 RI85 0.098 · 181.5, 기본) / cad_ri85(8개 RI85) — 어깨 구동기 팀장 확인 대기, actuator_params.json a2.case 로 전환
- actuator_params.json gravcomp.enable = true (함태훈 10/17 제안), actuatorfrcrange = forcerange
- meshes/visual · meshes/collision, URDF 메시 = ../meshes/... 상대 경로(strippath=false), 로더 하위 폴더 대응
- validate ②의 보상 없음 · A = gravcomp 뺀 모델(load_model strip_gravcomp) → 5종 통과 유지, render_v1 이중 보상 수정(11/11), 체크리스트 28/28
- a2_case_compare.py: case별 계단 응답 (yaw ω_n 140 → 35.8 rad/s)

Co-Authored-By: Claude Opus 5.5 <noreply@anthropic.com>
Claude-Session: https://claude.ai/code/session_01Xfhih1xrrj7ZVsqf6adRZk

File: b1/models/v1/urdf/b1_v1.urdf (robot description, URDF)
Before this commit: robot b1_v1, 17 links, 16 joints
Links:
- link left_elbow_link: geometry collision mesh filename=../meshes/collision/left_elbow_link_collision.stl; visual mesh filename=../meshes/visual/left_elbow_link_visual.stl
- link left_shoulder_pitch_link: geometry collision mesh filename=../meshes/collision/left_shoulder_pitch_link_collision.stl; visual mesh filename=../meshes/visual/left_shoulder_pitch_link_visual.stl
- link left_shoulder_roll_link: geometry collision mesh filename=../meshes/collision/left_shoulder_roll_link_collision.stl; visual mesh filename=../meshes/visual/left_shoulder_roll_link_visual.stl
- link left_shoulder_yaw_link: geometry collision mesh filename=../meshes/collision/left_shoulder_yaw_link_collision.stl; visual mesh filename=../meshes/visual/left_shoulder_yaw_link_visual.stl
- link right_elbow_link: geometry collision mesh filename=../meshes/collision/right_elbow_link_collision.stl; visual mesh filename=../meshes/visual/right_elbow_link_visual.stl
- link right_shoulder_pitch_link: geometry collision mesh filename=../meshes/collision/right_shoulder_pitch_link_collision.stl; visual mesh filename=../meshes/visual/right_shoulder_pitch_link_visual.stl
- link right_shoulder_roll_link: geometry collision mesh filename=../meshes/collision/right_shoulder_roll_link_collision.stl; visual mesh filename=../meshes/visual/right_shoulder_roll_link_visual.stl
- link right_shoulder_yaw_link: geometry collision mesh filename=../meshes/collision/right_shoulder_yaw_link_collision.stl; visual mesh filename=../meshes/visual/right_shoulder_yaw_link_visual.stl
- link torso_link: geometry collision box size=0.12 0.15 0.85; collision mesh filename=../meshes/collision/torso_link_collision.stl
Joints:
- joint left_elbow_joint: limit lower=-1.83 upper=1.83 effort=100.0 velocity=3.0 -> lower=-1.83 upper=1.83 effort=181.5 velocity=3.0
- joint left_shoulder_pitch_joint: limit lower=-3.0 upper=3.0 effort=100.0 velocity=3.0 -> lower=-3.0 upper=3.0 effort=381.7 velocity=3.0
- joint left_shoulder_roll_joint: limit lower=-0.28 upper=1.5 effort=100.0 velocity=3.0 -> lower=-0.28 upper=1.5 effort=381.7 velocity=3.0
- joint left_shoulder_yaw_joint: limit lower=-2.5 upper=2.5 effort=100.0 velocity=3.0 -> lower=-2.5 upper=2.5 effort=381.7 velocity=3.0
- joint right_elbow_joint: limit lower=-1.83 upper=1.83 effort=100.0 velocity=3.0 -> lower=-1.83 upper=1.83 effort=181.5 velocity=3.0
- joint right_shoulder_pitch_joint: limit lower=-3.0 upper=3.0 effort=100.0 velocity=3.0 -> lower=-3.0 upper=3.0 effort=381.7 velocity=3.0
- joint right_shoulder_roll_joint: limit lower=-0.28 upper=1.5 effort=100.0 velocity=3.0 -> lower=-0.28 upper=1.5 effort=381.7 velocity=3.0
- joint right_shoulder_yaw_joint: limit lower=-2.5 upper=2.5 effort=100.0 velocity=3.0 -> lower=-2.5 upper=2.5 effort=381.7 velocity=3.0

File: b1/models/v1/urdf/b1_v1_isaac.urdf (robot description, URDF)
Before this commit: robot b1_v1_isaac, 19 links, 18 joints
Links:
- link left_elbow_link: geometry collision mesh filename=../meshes/collision/left_elbow_link_collision.stl; visual mesh filename=../meshes/visual/left_elbow_link_visual.stl
- link left_shoulder_pitch_link: geometry collision mesh filename=../meshes/collision/left_shoulder_pitch_link_collision.stl; visual mesh filename=../meshes/visual/left_shoulder_pitch_link_visual.stl
- link left_shoulder_roll_link: geometry collision mesh filename=../meshes/collision/left_shoulder_roll_link_collision.stl; visual mesh filename=../meshes/visual/left_shoulder_roll_link_visual.stl
- link left_shoulder_yaw_link: geometry collision mesh filename=../meshes/collision/left_shoulder_yaw_link_collision.stl; visual mesh filename=../meshes/visual/left_shoulder_yaw_link_visual.stl
- link right_elbow_link: geometry collision mesh filename=../meshes/collision/right_elbow_link_collision.stl; visual mesh filename=../meshes/visual/right_elbow_link_visual.stl
- link right_shoulder_pitch_link: geometry collision mesh filename=../meshes/collision/right_shoulder_pitch_link_collision.stl; visual mesh filename=../meshes/visual/right_shoulder_pitch_link_visual.stl
- link right_shoulder_roll_link: geometry collision mesh filename=../meshes/collision/right_shoulder_roll_link_collision.stl; visual mesh filename=../meshes/visual/right_shoulder_roll_link_visual.stl
- link right_shoulder_yaw_link: geometry collision mesh filename=../meshes/collision/right_shoulder_yaw_link_collision.stl; visual mesh filename=../meshes/visual/right_shoulder_yaw_link_visual.stl
- link torso_link: geometry collision box size=0.12 0.15 0.85; collision mesh filename=../meshes/collision/torso_link_collision.stl
Joints:
- joint left_elbow_joint: limit lower=-1.83 upper=1.83 effort=100.0 velocity=3.0 -> lower=-1.83 upper=1.83 effort=181.5 velocity=3.0
- joint left_shoulder_pitch_joint: limit lower=-3.0 upper=3.0 effort=100.0 velocity=3.0 -> lower=-3.0 upper=3.0 effort=381.7 velocity=3.0
- joint left_shoulder_roll_joint: limit lower=-0.28 upper=1.5 effort=100.0 velocity=3.0 -> lower=-0.28 upper=1.5 effort=381.7 velocity=3.0
- joint left_shoulder_yaw_joint: limit lower=-2.5 upper=2.5 effort=100.0 velocity=3.0 -> lower=-2.5 upper=2.5 effort=381.7 velocity=3.0
- joint right_elbow_joint: limit lower=-1.83 upper=1.83 effort=100.0 velocity=3.0 -> lower=-1.83 upper=1.83 effort=181.5 velocity=3.0
- joint right_shoulder_pitch_joint: limit lower=-3.0 upper=3.0 effort=100.0 velocity=3.0 -> lower=-3.0 upper=3.0 effort=381.7 velocity=3.0
- joint right_shoulder_roll_joint: limit lower=-0.28 upper=1.5 effort=100.0 velocity=3.0 -> lower=-0.28 upper=1.5 effort=381.7 velocity=3.0
- joint right_shoulder_yaw_joint: limit lower=-2.5 upper=2.5 effort=100.0 velocity=3.0 -> lower=-2.5 upper=2.5 effort=381.7 velocity=3.0
